File: PowerSwap.sch (KiCad schematic (older format))
At the start: 10 parts

Commit message: Added values to schematic and added inductor footprint
Parts:
- added C?: 0.1UF, symbol C
- added R?: 0, symbol R
- 2.2u: renamed from L?; Link (none) -> http://parts.io/detail/2903506/LQH3NPN2R2MM0L; MPN (none) -> LQH3NPN2R2MM0L
- C?: value C -> 4.7UF
- C?: value C -> 22UF
- R?: value R -> 1.2M
- R?: value R -> 215K
Connections:
- net Earth: now also C?.2
- net at C?.1, P?.2 (P2), U?.5 (VIN): now also R?.2; no longer R?.2, R?.2, U?.8 (VINA)
- new net: C?.1, R?.1, R?.2, R?.2, U?.8 (VINA)
Changed lines of the file:
@@
 $EndComp
 $Comp
-L INDUCTOR L?
+L INDUCTOR 2.2u
 U 1 1 55BC16C0
 P 5600 2250
-F 0 "L?" V 5550 2250 50  0000 C CNN
+F 0 "2.2u" V 5550 2250 50  0000 C CNN
 F 1 "INDUCTOR" V 5700 2250 50  0000 C CNN
 F 2 "" H 5600 2250 60  0000 C CNN
 F 3 "" H 5600 2250 60  0000 C CNN
+F 4 "LQH3NPN2R2MM0L" V 5600 2250 60  0001 C CNN "MPN"
+F 5 "http://parts.io/detail/2903506/LQH3NPN2R2MM0L" V 5600 2250 60  0001 C CNN "Link"
 	1    5600 2250
 	0    -1   -1   0
@@
 P 2800 3300
 F 0 "C?" H 2825 3400 50  0000 L CNN
-F 1 "C" H 2825 3200 50  0000 L CNN
+F 1 "4.7UF" H 2825 3200 50  0000 L CNN
 F 2 "" H 2838 3150 30  0000 C CNN
 F 3 "" H 2800 3300 60  0000 C CNN
@@
 P 7950 3350
 F 0 "C?" H 7975 3450 50  0000 L CNN
-F 1 "C" H 7975 3250 50  0000 L CNN
+F 1 "22UF" H 7975 3250 50  0000 L CNN
 F 2 "" H 7988 3200 30  0000 C CNN
 F 3 "" H 7950 3350 60  0000 C CNN
@@
 P 7350 3350
 F 0 "R?" V 7430 3350 50  0000 C CNN
-F 1 "R" V 7350 3350 50  0000 C CNN
+F 1 "1.2M" V 7350 3350 50  0000 C CNN
 F 2 "" V 7280 3350 30  0000 C CNN
 F 3 "" H 7350 3350 30  0000 C CNN
@@
 P 7350 3850
 F 0 "R?" V 7430 3850 50  0000 C CNN
-F 1 "R" V 7350 3850 50  0000 C CNN
+F 1 "215K" V 7350 3850 50  0000 C CNN
 F 2 "" V 7280 3850 30  0000 C CNN
 F 3 "" H 7350 3850 30  0000 C CNN
@@
 	2800 3100 2800 3150
 Wire Wire Line
-	4900 3250 4650 3250
-Wire Wire Line
-	4650 3250 4650 3100
-Connection ~ 4650 3100
+	3850 3250 4900 3250
 $Comp
 L R R?
@@
 	4900 3400 4750 3400
 Wire Wire Line
-	4450 3400 4300 3400
-Wire Wire Line
-	4300 3400 4300 3100
-Connection ~ 4300 3100
+	4050 3400 4450 3400
 Wire Wire Line
 	4900 3550 4500 3550
 Wire Wire Line
 	4200 3550 4050 3550
-Wire Wire Line
-	4050 3550 4050 3100
-Connection ~ 4050 3100
 Wire Wire Line
 	4600 2850 4600 2250
@@
 	2300 3550 2800 3550
 Connection ~ 2800 3550
+$Comp
+L R R?
+U 1 1 55C689AF
+P 3700 3250
+F 0 "R?" V 3780 3250 50  0000 C CNN
+F 1 "0" V 3700 3250 50  0000 C CNN
+F 2 "" V 3630 3250 30  0000 C CNN
+F 3 "" H 3700 3250 30  0000 C CNN
+	1    3700 3250
+	0    1    1    0
+$EndComp
+Wire Wire Line
+	4050 3250 4050 3600
+Connection ~ 4050 3400
+Connection ~ 4050 3250
+Wire Wire Line
+	3550 3250 3450 3250
+Wire Wire Line
+	3450 3250 3450 3100
+Connection ~ 3450 3100
+$Comp
+L C C?
+U 1 1 55C68B85
+P 4050 3750
+F 0 "C?" H 4075 3850 50  0000 L CNN
+F 1 "0.1UF" H 4075 3650 50  0000 L CNN
+F 2 "" H 4088 3600 30  0000 C CNN
+F 3 "" H 4050 3750 60  0000 C CNN
+	1    4050 3750
+	1    0    0    -1
+$EndComp
+Connection ~ 4050 3550
+Wire Wire Line
+	4050 3900 4050 4050
+$Comp
+L GNDPWR #PWR?
+U 1 1 55C68C50
+P 4050 4050
+F 0 "#PWR?" H 4050 3850 50  0001 C CNN
+F 1 "GNDPWR" H 4050 3920 50  0000 C CNN
+F 2 "" H 4050 4000 60  0000 C CNN
+F 3 "" H 4050 4000 60  0000 C CNN
+	1    4050 4050
+	1    0    0    -1
+$EndComp
 $EndSCHEMATC

Commit message: Imported footprints
Parts:
- added P? (x4): TST, symbol TST
- L1: renamed from 2.2u; value INDUCTOR -> 2.2uH
- gave numbers to parts that had none: 8
Connections:
- net Earth: now also P?.1
- net VOUT: now reaches C2.1, P2.1 (P1), R1.1, U1.1 (VOUT)
- net VOUT: now also P?.1
- net FB: now reaches R1.2, R2.1, U1.10 (FB)
- net FB: now also P?.1
- net VIN: now reaches C1.1, P1.2 (P2), R?.2, U1.5 (VIN)
- net VIN: now also P?.1
- net VINA: now reaches C3.1, R?.1, R?.2, R?.2, U1.8 (VINA)
Changed lines of the file:
@@
 $EndDescr
 $Comp
-L TPS63030 U?
+L TPS63030 U1
 U 1 1 55BC1656
 P 5600 3400
-F 0 "U?" H 6000 2850 60  0000 C CNN
+F 0 "U1" H 6000 2850 60  0000 C CNN
 F 1 "TPS63030" H 5600 4100 60  0000 C CNN
 F 2 "" H 5550 3500 60  0000 C CNN
@@
 $EndComp
 $Comp
-L INDUCTOR 2.2u
+L INDUCTOR L1
 U 1 1 55BC16C0
 P 5600 2250
-F 0 "2.2u" V 5550 2250 50  0000 C CNN
-F 1 "INDUCTOR" V 5700 2250 50  0000 C CNN
+F 0 "L1" V 5550 2250 50  0000 C CNN
+F 1 "2.2uH" V 5700 2250 50  0000 C CNN
 F 2 "" H 5600 2250 60  0000 C CNN
 F 3 "" H 5600 2250 60  0000 C CNN
@@
 $EndComp
 $Comp
-L C C?
+L C C1
 U 1 1 55BC171B
 P 2800 3300
-F 0 "C?" H 2825 3400 50  0000 L CNN
+F 0 "C1" H 2825 3400 50  0000 L CNN
 F 1 "4.7UF" H 2825 3200 50  0000 L CNN
 F 2 "" H 2838 3150 30  0000 C CNN
@@
 $EndComp
 $Comp
-L C C?
+L C C2
 U 1 1 55BC18FD
 P 7950 3350
-F 0 "C?" H 7975 3450 50  0000 L CNN
+F 0 "C2" H 7975 3450 50  0000 L CNN
 F 1 "22UF" H 7975 3250 50  0000 L CNN
 F 2 "" H 7988 3200 30  0000 C CNN
@@
 $EndComp
 $Comp
-L R R?
+L R R1
 U 1 1 55BC195F
 P 7350 3350
-F 0 "R?" V 7430 3350 50  0000 C CNN
+F 0 "R1" V 7430 3350 50  0000 C CNN
 F 1 "1.2M" V 7350 3350 50  0000 C CNN
 F 2 "" V 7280 3350 30  0000 C CNN
@@
 $EndComp
 $Comp
-L R R?
+L R R2
 U 1 1 55BC19CB
 P 7350 3850
-F 0 "R?" V 7430 3850 50  0000 C CNN
+F 0 "R2" V 7430 3850 50  0000 C CNN
 F 1 "215K" V 7350 3850 50  0000 C CNN
 F 2 "" V 7280 3850 30  0000 C CNN
@@
 $EndComp
 Wire Wire Line
-	6250 3800 6450 3800
+	6250 3800 6600 3800
 Wire Wire Line
 	6450 3800 6450 4050
@@
 Connection ~ 7950 3100
 $Comp
-L CONN_01X02 P?
+L CONN_01X02 P2
 U 1 1 55BC233B
 P 9000 3150
-F 0 "P?" H 9000 3300 50  0000 C CNN
+F 0 "P2" H 9000 3300 50  0000 C CNN
 F 1 "CONN_01X02" V 9100 3150 50  0000 C CNN
 F 2 "" H 9000 3150 60  0000 C CNN
@@
 Connection ~ 7950 3600
 $Comp
-L CONN_01X02 P?
+L CONN_01X02 P1
 U 1 1 55BC241B
 P 1850 3150
-F 0 "P?" H 1850 3300 50  0000 C CNN
+F 0 "P1" H 1850 3300 50  0000 C CNN
 F 1 "CONN_01X02" V 1950 3150 50  0000 C CNN
 F 2 "" H 1850 3150 60  0000 C CNN
@@
 Connection ~ 3450 3100
 $Comp
-L C C?
+L C C3
 U 1 1 55C68B85
 P 4050 3750
-F 0 "C?" H 4075 3850 50  0000 L CNN
+F 0 "C3" H 4075 3850 50  0000 L CNN
 F 1 "0.1UF" H 4075 3650 50  0000 L CNN
 F 2 "" H 4088 3600 30  0000 C CNN
@@
 	1    0    0    -1
 $EndComp
+$Comp
+L TST P?
+U 1 1 55C6D252
+P 4050 2950
+F 0 "P?" H 4050 3250 50  0000 C BNN
+F 1 "TST" H 4050 3200 50  0000 C CNN
+F 2 "" H 4050 2950 60  0000 C CNN
+F 3 "" H 4050 2950 60  0000 C CNN
+	1    4050 2950
+	1    0    0    -1
+$EndComp
+$Comp
+L TST P?
+U 1 1 55C6D6B9
+P 7100 3500
+F 0 "P?" H 7100 3800 50  0000 C BNN
+F 1 "TST" H 7100 3750 50  0000 C CNN
+F 2 "" H 7100 3500 60  0000 C CNN
+F 3 "" H 7100 3500 60  0000 C CNN
+	1    7100 3500
+	1    0    0    -1
+$EndComp
+$Comp
+L TST P?
+U 1 1 55C6D735
+P 6600 3800
+F 0 "P?" H 6600 4100 50  0000 C BNN
+F 1 "TST" H 6600 4050 50  0000 C CNN
+F 2 "" H 6600 3800 60  0000 C CNN
+F 3 "" H 6600 3800 60  0000 C CNN
+	1    6600 3800
+	1    0    0    -1
+$EndComp
+$Comp
+L TST P?
+U 1 1 55C6D790
+P 7700 3050
+F 0 "P?" H 7700 3350 50  0000 C BNN
+F 1 "TST" H 7700 3300 50  0000 C CNN
+F 2 "" H 7700 3050 60  0000 C CNN
+F 3 "" H 7700 3050 60  0000 C CNN
+	1    7700 3050
+	1    0    0    -1
+$EndComp
+Wire Wire Line
+	4050 2950 4050 3100
+Connection ~ 4050 3100
+Wire Wire Line
+	7700 3100 7700 3050
+Connection ~ 7700 3100
+Wire Wire Line
+	7100 3500 7100 3600
+Connection ~ 7100 3600
+Connection ~ 6450 3800
+Text Label 4500 3100 0    60   ~ 0
+VIN
+Text Label 4500 3250 0    60   ~ 0
+VINA
+Text Label 6350 3100 0    60   ~ 0
+VOUT
+Text Label 6400 3450 0    60   ~ 0
+FB
 $EndSCHEMATC

Commit message: Finished Power Swap Layout
Parts:
- C1, C3: footprint (none) -> Capacitors_SMD:C_0805
- C2: footprint (none) -> Capacitors_SMD:C_1210
- L1: footprint (none) -> PowerSwap:LQH3NPN2R2MM0L
- P1, P2: footprint (none) -> Pin_Headers:Pin_Header_Straight_1x02
- P3, P4, P5, P6: renamed from P?; footprint (none) -> Measurement_Points:Measurement_Point_Square-SMD-Pad_Small
- R1, R2: footprint (none) -> Resistors_SMD:R_0805
- R3, R4, R5: renamed from R?; footprint (none) -> Resistors_SMD:R_0805
- U1: footprint (none) -> PowerSwap:TPS63030
Connections:
- net Earth: now also U1.11 (EP)
Changed lines of the file:
@@
 F 0 "U1" H 6000 2850 60  0000 C CNN
 F 1 "TPS63030" H 5600 4100 60  0000 C CNN
-F 2 "" H 5550 3500 60  0000 C CNN
+F 2 "PowerSwap:TPS63030" H 5550 3500 60  0001 C CNN
 F 3 "" H 5550 3500 60  0000 C CNN
 	1    5600 3400
@@
 F 0 "L1" V 5550 2250 50  0000 C CNN
 F 1 "2.2uH" V 5700 2250 50  0000 C CNN
-F 2 "" H 5600 2250 60  0000 C CNN
+F 2 "PowerSwap:LQH3NPN2R2MM0L" H 5600 2250 60  0001 C CNN
 F 3 "" H 5600 2250 60  0000 C CNN
 F 4 "LQH3NPN2R2MM0L" V 5600 2250 60  0001 C CNN "MPN"
@@
 F 0 "C1" H 2825 3400 50  0000 L CNN
 F 1 "4.7UF" H 2825 3200 50  0000 L CNN
-F 2 "" H 2838 3150 30  0000 C CNN
+F 2 "Capacitors_SMD:C_0805" H 2838 3150 30  0001 C CNN
 F 3 "" H 2800 3300 60  0000 C CNN
 	1    2800 3300
@@
 F 0 "C2" H 7975 3450 50  0000 L CNN
 F 1 "22UF" H 7975 3250 50  0000 L CNN
-F 2 "" H 7988 3200 30  0000 C CNN
+F 2 "Capacitors_SMD:C_1210" H 7988 3200 30  0001 C CNN
 F 3 "" H 7950 3350 60  0000 C CNN
 	1    7950 3350
@@
 F 0 "R1" V 7430 3350 50  0000 C CNN
 F 1 "1.2M" V 7350 3350 50  0000 C CNN
-F 2 "" V 7280 3350 30  0000 C CNN
+F 2 "Resistors_SMD:R_0805" V 7280 3350 30  0001 C CNN
 F 3 "" H 7350 3350 30  0000 C CNN
 	1    7350 3350
@@
 F 0 "R2" V 7430 3850 50  0000 C CNN
 F 1 "215K" V 7350 3850 50  0000 C CNN
-F 2 "" V 7280 3850 30  0000 C CNN
+F 2 "Resistors_SMD:R_0805" V 7280 3850 30  0001 C CNN
 F 3 "" H 7350 3850 30  0000 C CNN
 	1    7350 3850
@@
 $EndComp
 $Comp
-L Earth #PWR?
+L Earth #PWR01
 U 1 1 55BC1A42
 P 4550 4050
-F 0 "#PWR?" H 4550 3800 50  0001 C CNN
+F 0 "#PWR01" H 4550 3800 50  0001 C CNN
 F 1 "Earth" H 4550 3900 50  0001 C CNN
 F 2 "" H 4550 4050 60  0000 C CNN
@@
 $EndComp
 $Comp
-L GNDPWR #PWR?
+L GNDPWR #PWR02
 U 1 1 55BC1A98
 P 4750 4050
-F 0 "#PWR?" H 4750 3850 50  0001 C CNN
+F 0 "#PWR02" H 4750 3850 50  0001 C CNN
 F 1 "GNDPWR" H 4750 3920 50  0000 C CNN
 F 2 "" H 4750 4000 60  0000 C CNN
@@
 Connection ~ 4750 3800
 $Comp
-L GNDPWR #PWR?
+L GNDPWR #PWR03
 U 1 1 55BC1B2E
 P 6450 4050
-F 0 "#PWR?" H 6450 3850 50  0001 C CNN
+F 0 "#PWR03" H 6450 3850 50  0001 C CNN
 F 1 "GNDPWR" H 6450 3920 50  0000 C CNN
 F 2 "" H 6450 4000 60  0000 C CNN
@@
 	7350 4000 7350 4150
 $Comp
-L GNDPWR #PWR?
+L GNDPWR #PWR04
 U 1 1 55BC1BC4
 P 7350 4150
-F 0 "#PWR?" H 7350 3950 50  0001 C CNN
+F 0 "#PWR04" H 7350 3950 50  0001 C CNN
 F 1 "GNDPWR" H 7350 4020 50  0000 C CNN
 F 2 "" H 7350 4100 60  0000 C CNN
@@
 $EndComp
 $Comp
-L GNDPWR #PWR?
+L GNDPWR #PWR05
 U 1 1 55BC1BDB
 P 7950 3650
-F 0 "#PWR?" H 7950 3450 50  0001 C CNN
+F 0 "#PWR05" H 7950 3450 50  0001 C CNN
 F 1 "GNDPWR" H 7950 3520 50  0000 C CNN
 F 2 "" H 7950 3600 60  0000 C CNN
@@
 Connection ~ 7350 3100
 $Comp
-L GNDPWR #PWR?
+L GNDPWR #PWR06
 U 1 1 55BC1CD6
 P 2800 3600
-F 0 "#PWR?" H 2800 3400 50  0001 C CNN
+F 0 "#PWR06" H 2800 3400 50  0001 C CNN
 F 1 "GNDPWR" H 2800 3470 50  0000 C CNN
 F 2 "" H 2800 3550 60  0000 C CNN
@@
 	3850 3250 4900 3250
 $Comp
-L R R?
+L R R5
 U 1 1 55BC1DB4
 P 4600 3400
-F 0 "R?" V 4680 3400 50  0000 C CNN
+F 0 "R5" V 4680 3400 50  0000 C CNN
 F 1 "0" V 4600 3400 50  0000 C CNN
-F 2 "" V 4530 3400 30  0000 C CNN
+F 2 "Resistors_SMD:R_0805" V 4530 3400 30  0001 C CNN
 F 3 "" H 4600 3400 30  0000 C CNN
 	1    4600 3400
@@
 $EndComp
 $Comp
-L R R?
+L R R4
 U 1 1 55BC1E39
 P 4350 3550
-F 0 "R?" V 4430 3550 50  0000 C CNN
+F 0 "R4" V 4430 3550 50  0000 C CNN
 F 1 "0" V 4350 3550 50  0000 C CNN
-F 2 "" V 4280 3550 30  0000 C CNN
+F 2 "Resistors_SMD:R_0805" V 4280 3550 30  0001 C CNN
 F 3 "" H 4350 3550 30  0000 C CNN
 	1    4350 3550
@@
 F 0 "P2" H 9000 3300 50  0000 C CNN
 F 1 "CONN_01X02" V 9100 3150 50  0000 C CNN
-F 2 "" H 9000 3150 60  0000 C CNN
+F 2 "Pin_Headers:Pin_Header_Straight_1x02" H 9000 3150 60  0001 C CNN
 F 3 "" H 9000 3150 60  0000 C CNN
 	1    9000 3150
@@
 F 0 "P1" H 1850 3300 50  0000 C CNN
 F 1 "CONN_01X02" V 1950 3150 50  0000 C CNN
-F 2 "" H 1850 3150 60  0000 C CNN
+F 2 "Pin_Headers:Pin_Header_Straight_1x02" H 1850 3150 60  0001 C CNN
 F 3 "" H 1850 3150 60  0000 C CNN
 	1    1850 3150
@@
 Connection ~ 2800 3550
 $Comp
-L R R?
+L R R3
 U 1 1 55C689AF
 P 3700 3250
-F 0 "R?" V 3780 3250 50  0000 C CNN
+F 0 "R3" V 3780 3250 50  0000 C CNN
 F 1 "0" V 3700 3250 50  0000 C CNN
-F 2 "" V 3630 3250 30  0000 C CNN
+F 2 "Resistors_SMD:R_0805" V 3630 3250 30  0001 C CNN
 F 3 "" H 3700 3250 30  0000 C CNN
 	1    3700 3250
@@
 F 0 "C3" H 4075 3850 50  0000 L CNN
 F 1 "0.1UF" H 4075 3650 50  0000 L CNN
-F 2 "" H 4088 3600 30  0000 C CNN
+F 2 "Capacitors_SMD:C_0805" H 4088 3600 30  0001 C CNN
 F 3 "" H 4050 3750 60  0000 C CNN
 	1    4050 3750
@@
 	4050 3900 4050 4050
 $Comp
-L GNDPWR #PWR?
+L GNDPWR #PWR07
 U 1 1 55C68C50
 P 4050 4050
-F 0 "#PWR?" H 4050 3850 50  0001 C CNN
+F 0 "#PWR07" H 4050 3850 50  0001 C CNN
 F 1 "GNDPWR" H 4050 3920 50  0000 C CNN
 F 2 "" H 4050 4000 60  0000 C CNN
@@
 $EndComp
 $Comp
-L TST P?
+L TST P3
 U 1 1 55C6D252
 P 4050 2950
-F 0 "P?" H 4050 3250 50  0000 C BNN
+F 0 "P3" H 4050 3250 50  0000 C BNN
 F 1 "TST" H 4050 3200 50  0000 C CNN
-F 2 "" H 4050 2950 60  0000 C CNN
+F 2 "Measurement_Points:Measurement_Point_Square-SMD-Pad_Small" H 4050 2950 60  0001 C CNN
 F 3 "" H 4050 2950 60  0000 C CNN
 	1    4050 2950
@@
 $EndComp
 $Comp
-L TST P?
+L TST P5
 U 1 1 55C6D6B9
 P 7100 3500
-F 0 "P?" H 7100 3800 50  0000 C BNN
+F 0 "P5" H 7100 3800 50  0000 C BNN
 F 1 "TST" H 7100 3750 50  0000 C CNN
-F 2 "" H 7100 3500 60  0000 C CNN
+F 2 "Measurement_Points:Measurement_Point_Square-SMD-Pad_Small" H 7100 3500 60  0001 C CNN
 F 3 "" H 7100 3500 60  0000 C CNN
 	1    7100 3500
@@
 $EndComp
 $Comp
-L TST P?
+L TST P4
 U 1 1 55C6D735
 P 6600 3800
-F 0 "P?" H 6600 4100 50  0000 C BNN
+F 0 "P4" H 6600 4100 50  0000 C BNN
 F 1 "TST" H 6600 4050 50  0000 C CNN
-F 2 "" H 6600 3800 60  0000 C CNN
+F 2 "Measurement_Points:Measurement_Point_Square-SMD-Pad_Small" H 6600 3800 60  0001 C CNN
 F 3 "" H 6600 3800 60  0000 C CNN
 	1    6600 3800
@@
 $EndComp
 $Comp
-L TST P?
+L TST P6
 U 1 1 55C6D790
 P 7700 3050
-F 0 "P?" H 7700 3350 50  0000 C BNN
+F 0 "P6" H 7700 3350 50  0000 C BNN
 F 1 "TST" H 7700 3300 50  0000 C CNN
-F 2 "" H 7700 3050 60  0000 C CNN
+F 2 "Measurement_Points:Measurement_Point_Square-SMD-Pad_Small" H 7700 3050 60  0001 C CNN
 F 3 "" H 7700 3050 60  0000 C CNN
 	1    7700 3050
@@
 Text Label 6400 3450 0    60   ~ 0
 FB
+Wire Wire Line
+	5600 4100 4950 4100
+Wire Wire Line
+	4950 4100 4950 3900
+Wire Wire Line
+	4950 3900 4750 3900
+Connection ~ 4750 3900
+Wire Wire Line
+	5500 4100 5500 4250
+Wire Wire Line
+	5500 4250 6300 4250
+Wire Wire Line
+	6300 4250 6300 3800
+Connection ~ 6300 3800
+Connection ~ 5500 4100
 $EndSCHEMATC
